File: KiCad/WildlifeCapture.kicad_pcb (KiCad board)
At the start: 2 copper layers, 105 x 100 mm, 15 parts, among them P1 USB_A, P2 GPS, SW1 A, SW2 LEADSW, U1 IM920_interplan, U3 STM32F103C8T6MinimumDevelopBo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, U4 RASPBERRYPI_GPIO_40

Commit message: Change to Take 2
Parts:
- removed P1: USB_A, Connect:USB_A
- added BT3: Battery, library:18650BatteryCase, F.Cu at (134.1, 103.2)
- added C1: CP1, Capacitors_ThroughHole:C_Radial_D10_L13_P5, F.Cu at (158.2, 78.7)
- added J1: DCJACK, library:DCJACK, F.Cu at (95.1, 149.2)
- added P3: EN, Pin_Headers:Pin_Header_Straight_1x01, F.Cu at (102.7, 70.2)
- added P4: NanoPi_USB/Audio/IR, Pin_Headers:Pin_Header_Straight_1x12, B.Cu at (135.1, 74.7)
- added P5: USB_A, Connect:USB_A_Vertical, F.Cu at (148.0, 88.2)
- added P6: USB_A, Connect:USB_A_Vertical, F.Cu at (95.9, 118.7)
- added P7: SERVICE, Pin_Headers:Pin_Header_Straight_1x04, F.Cu at (165.8, 86.3)
- added P8: VCC, Pin_Headers:Pin_Header_Straight_1x04, F.Cu at (165.8, 88.9)
- added P9: GND, Pin_Headers:Pin_Header_Straight_1x04, F.Cu at (165.8, 91.4)
- added R1: R, Discret:R4, F.Cu at (107.4, 60.9)
- added R5: R, Discret:R4, F.Cu at (112.1, 44.5)
- added SP1: SPEAKER, Buzzers_Beepers:MagneticBuzzer_ProSignal_ABT-410-RC, F.Cu at (146.4, 82.0)
- added SW3: SWITCH_INV, Buzzers_Beepers:Buzzer_12x9.5RM7.6, F.Cu at (97.2, 132.7)
- added U5: MT3608, library:MT3608, F.Cu at (120.1, 84.2)
- BT1: footprint Pin_Headers:Pin_Header_Straight_1x02 -> library:18650BatteryCase
- BT2: footprint library:BATTERY_CR2032_CH25-2032LF_CONFORTABLE -> library:18650BatteryCase
- U1, U4: moved to B.Cu
- moved D2 105.3 mm to (96.6, 137.8), turned to 0 degrees
- moved BT1 86.1 mm to (134.1, 124.7)
- moved U4 84.8 mm to (135.1, 40.2), turned to 90 degrees
- moved BT2 74.2 mm to (134.1, 146.2), turned to 0 degrees
- moved JP1 67.9 mm to (148.6, 70.4), turned to 270 degrees
- moved R4 60.1 mm to (145.9, 53.2)
- moved R3 56.5 mm to (145.7, 56.6), turned to 180 degrees
- moved U1 50.0 mm to (167.0, 71.1), turned to 180 degrees
- moved U3 47.2 mm to (99.7, 68.5), turned to 0 degrees
- moved P2 29.6 mm to (164.0, 78.1), turned to 90 degrees
- moved SW1 28.2 mm to (148.0, 41.2), turned to 270 degrees
- moved R2 27.9 mm to (137.3, 44.5)
- moved D1 24.8 mm to (140.6, 38.3), turned to 270 degrees
- moved SW2 7.44 mm to (124.1, 138.2)
Connections:
- net Net-(JP1-Pad2) renamed +5V
- D2 pad 1: Net-(BT1-Pad1) -> Net-(D2-Pad1)
- D2 pad 2: +3V3 -> +BATT
- JP1 pad 1: +3V3 -> +BATT
- R3 pad 1: +3V3 -> +BATT
- U1 pad 18: Net-(U1-Pad18) -> GND
- U1 pad 19: Net-(U1-Pad19) -> GND
- U1 pad 23: +3V3 -> +BATT
- U3 pad 14: Net-(U1-Pad6) -> Net-(U3-Pad14)
- U3 pad 15: Net-(U1-Pad7) -> Net-(U3-Pad15)
- U3 pad 20: +3V3 -> +BATT
- U3 pad 21: +3V3 -> Net-(BT1-Pad1)
- U3 pad 26: Net-(U3-Pad26) -> Net-(R2-Pad1)
- U3 pad 33: Net-(R2-Pad1) -> Net-(P7-Pad2)
- U3 pad 38: +3V3 -> +BATT
- U3 pad 6: Net-(U3-Pad6) -> Net-(U1-Pad6)
- U3 pad 7: Net-(P1-Pad3) -> Net-(U1-Pad7)
- U4 pad 17: Net-(U4-Pad17) -> +3V3
Routing:
- net +BATT: track 0.00 -> 263.7 mm, vias 0 -> 3
- net +3V3: track 249.8 -> 21.5 mm, vias 1 -> 0
- net GND: track 394.9 -> 601.9 mm, vias 1 -> 2
- net Net-(R2-Pad1): track 124.2 -> 7.64 mm
- net Net-(SW1-Pad2): track 124.8 -> 14.5 mm, vias 1 -> 0
- net Net-(BT1-Pad1): track 38.6 -> 142.7 mm, vias 0 -> 2
- net Net-(P4-Pad4): track 0.00 -> 81.9 mm, vias 0 -> 1
- net Net-(P4-Pad5): track 0.00 -> 78.7 mm, vias 0 -> 1
- net Net-(P7-Pad2): track 0.00 -> 77.0 mm, vias 0 -> 3
- net Net-(P7-Pad4): track 0.00 -> 76.9 mm, vias 0 -> 3
- net Net-(P7-Pad3): track 0.00 -> 75.7 mm, vias 0 -> 3
- net +5V: track 119.1 -> 194.3 mm, vias 0 -> 2
- net Net-(P7-Pad1): track 0.00 -> 74.6 mm, vias 0 -> 3
- net Net-(SW2-Pad1): track 33.9 -> 99.8 mm
- net Net-(U3-Pad8): track 54.1 -> 0.00 mm
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Other:
- board size 105 x 100 mm -> 90 x 120 mm
- board text added: "+ 18650 FeLiP0 -"
- board text added: "3V3 GND"
- board text added: "ENABLE"
- board text added: "IM920"
- board text added: "LEAD SW"
- board text added: "MT3608 Boost DCDC"
- board text added: "NanoPi"
- board text added: "NanoPi Neo"
- board text added: "PA1 PA0 PB7 PB6"
- board text added: "SERIAL"
- board text added: "SWITCH"

Commit message: Change to Take 3
Parts:
- added BT1: Battery, Pin_Headers:Pin_Header_Straight_1x02, F.Cu at (193.7, 76.8)
- added BT2: Battery, library:BATTERY_CR2032_CH25-2032LF_CONFORTABLE, B.Cu at (193.7, 75.8)
- added C1: C, Capacitors_SMD:C_1206, F.Cu at (201.5, 64.0)
- added D1: LED, LEDs:LED-5MM, F.Cu at (229.0, 57.3)
- added D2: DIODESCH, Diodes_SMD:MELF_Standard, F.Cu at (188.6, 97.8)
- added G***: AVTOKYO_10THLOGO, library:AVTOKYO_10THLOGO, B.Cu at (215.3, 120.6)
- added G***: AVTOKYOLOGO, AVTOKYO:AVTOKYOLOGO, F.Cu at (214.8, 162.3)
- added JP2: JUMPER3, Pin_Headers:Pin_Header_Straight_1x03, F.Cu at (132.1, 34.2)
- added JP3: JUMPER3, Pin_Headers:Pin_Header_Straight_1x03, F.Cu at (116.1, 34.2)
- added Q1: MOSFET_P, TO_SOT_Packages_SMD:SOT-23_Handsoldering, F.Cu at (104.8, 98.5)
- added R1: 10kΩ, Resistors_SMD:R_1206, F.Cu at (209.2, 64.0)
- added R2: 180Ω, Resistors_SMD:R_1206, F.Cu at (234.7, 66.6)
- added R3: 2.7kΩ, Resistors_SMD:R_1206, F.Cu at (216.6, 132.0)
- added R4: OPEN, Discret:R4, F.Cu at (216.6, 129.5)
- added SP1: SPEAKER, Buzzers_Beepers:MagneticBuzzer_ProSignal_ABT-410-RC, F.Cu at (215.3, 147.3)
- added SW1: A, Buttons_Switches_SMD:SW_SPST_EVPBF, F.Cu at (238.2, 133.3)
- added SW2: B, Buttons_Switches_SMD:SW_SPST_EVPBF, F.Cu at (229.3, 138.4)
- added SW3: UP, Buttons_Switches_SMD:SW_SPST_EVPBF, F.Cu at (197.5, 130.8)
- added SW4: DOWN, Buttons_Switches_SMD:SW_SPST_EVPBF, F.Cu at (197.5, 143.5)
- added SW5: LEFT, Buttons_Switches_SMD:SW_SPST_EVPBF, F.Cu at (203.9, 137.1)
- added SW6: RIGHT, Buttons_Switches_SMD:SW_SPST_EVPBF, F.Cu at (191.2, 137.1)
- added U1: PhotoReciever_GP1USC4XQS_SHARP, Pin_Headers:Pin_Header_Straight_1x03, F.Cu at (202.6, 57.1)
- added U2: OLED_0.96in_SPI, library:OLED_0.96in_SPI, F.Cu at (215.3, 92.7)
- added U3: STM32F103C8T6MinimumDevelopBoard, library:STM32F103C8T6ARMMiniSystemDevboard_RobotDyn, F.Cu at (242.0, 102.8)
- added U6: ES920LR_LPWA_EASEL, library:ES920_LPWA_EASEL, F.Cu at (172.1, 47.2)
- added W1: TEST_1P, Pin_Headers:Pin_Header_Straight_1x01, F.Cu at (159.1, 39.2)
- added W2: TEST_1P, Pin_Headers:Pin_Header_Straight_1x01, F.Cu at (161.1, 43.2)
- added W3: TEST_1P, Pin_Headers:Pin_Header_Straight_1x01, F.Cu at (166.1, 60.2)
- moved R1 38.7 mm to (113.7, 99.0), turned to 0 degrees
- moved BT3 11.0 mm to (134.1, 114.2)
- moved BT1 10.0 mm to (134.1, 134.7)
- moved BT2 10.0 mm to (134.1, 156.2)
- moved D2 10.0 mm to (96.6, 147.8)
- moved J1 10.0 mm to (95.1, 159.2)
- moved P6 10.0 mm to (95.9, 128.7)
- moved SW2 10.0 mm to (124.1, 148.2)
- moved SW3 10.0 mm to (97.2, 142.7)
Connections:
- R1 pad 1: Net-(P3-Pad1) -> Net-(Q1-PadG)
- R1 pad 2: GND -> +BATT
- U1 pad 6: Net-(U1-Pad6) -> Net-(JP2-Pad1)
- U1 pad 7: Net-(U1-Pad7) -> Net-(JP2-Pad3)
- U3 pad 4: Net-(P3-Pad1) -> Net-(Q1-PadG)
- U3 pad 6: Net-(U1-Pad6) -> Net-(JP2-Pad1)
- U3 pad 7: Net-(U1-Pad7) -> Net-(JP2-Pad3)
- U4 pad 10: Net-(U1-Pad7) -> Net-(JP3-Pad2)
- U4 pad 8: Net-(U1-Pad6) -> Net-(JP2-Pad2)
- U5 pad 1: +BATT -> Net-(Q1-PadS)
Routing:
- net GND: track 601.9 -> 928.7 mm
- net +3V3: track 21.5 -> 197.0 mm, vias 0 -> 3
- net Net-(JP2-Pad3): track 0.00 -> 140.3 mm, vias 0 -> 3
- net Net-(JP2-Pad1): track 0.00 -> 135.1 mm, vias 0 -> 3
- net Net-(SP1-Pad2): track 27.5 -> 147.8 mm, vias 1 -> 2
- net Net-(SW3-Pad2): track 0.00 -> 119.8 mm, vias 0 -> 1
- net Net-(U2-Pad5): track 0.00 -> 118.2 mm
- net Net-(R1-Pad1): track 0.00 -> 118.0 mm, vias 0 -> 1
- net Net-(U2-Pad7): track 0.00 -> 115.2 mm, vias 0 -> 1
- net Net-(U3-Pad1): track 0.00 -> 114.7 mm
- net Net-(R3-Pad2): track 115.0 -> 229.1 mm, vias 0 -> 3
- net Net-(U2-Pad3): track 0.00 -> 114.1 mm
- net Net-(U2-Pad6): track 0.00 -> 111.2 mm, vias 0 -> 1
- net Net-(U2-Pad4): track 0.00 -> 109.4 mm, vias 0 -> 1
- net Net-(R2-Pad1): track 7.64 -> 109.1 mm, vias 0 -> 2
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Other:
- board size 90 x 120 mm -> 157.1 x 135.1 mm
