File: KiCad/WildlifeCapture.sch (KiCad schematic (older format))
At the start: 17 parts, among them P1 USB_A, P2 GPS, SW1 A, SW2 LEADSW, U1 IM920_interplan, U2 OLED_0.96in_I2C, U3 STM32F103C8T6MinimumDevelopBo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, U4 RASPBERRYPI_GPIO_40

Commit message: Change to Take 2
Parts:
- removed P1: USB_A, Connect:USB_A, symbol USB_A
- added BT3: Battery, library:18650BatteryCase, symbol Battery
- added C1: CP1, Capacitors_ThroughHole:C_Radial_D10_L13_P5, symbol CP1
- added J1: DCJACK, library:DCJACK, symbol DCJACK
- added P3: EN, Pin_Headers:Pin_Header_Straight_1x01, symbol CONN_01X01
- added P4: NanoPi_USB/Audio/IR, Pin_Headers:Pin_Header_Straight_1x12, symbol NanoPi_USB/Audio/IR
- added P5, P6: USB_A, Connect:USB_A_Vertical, symbol USB_A
- added P7: SERVICE, Pin_Headers:Pin_Header_Straight_1x04, symbol CONN_01X04
- added P8: VCC, Pin_Headers:Pin_Header_Straight_1x04, symbol CONN_01X04
- added P9: GND, Pin_Headers:Pin_Header_Straight_1x04, symbol CONN_01X04
- added R1, R5: R, Discret:R4, symbol R
- added SW3: SWITCH_INV, Buzzers_Beepers:Buzzer_12x9.5RM7.6, symbol SWITCH_INV
- added U5: MT3608, library:MT3608, symbol MT3608
- BT1: footprint Pin_Headers:Pin_Header_Straight_1x02 -> library:18650BatteryCase
- BT2: footprint library:BATTERY_CR2032_CH25-2032LF_CONFORTABLE -> library:18650BatteryCase
Connections:
- net +3V3: now also U4.17 (3.3V); no longer D2.2 (K), JP1.1, R3.1, U1.23 (VCC), U3.20 (3.3V), U3.21 (VBAT), U3.38 (3.3V)
- net GND: now also U1.18 (MODE2), U1.19 (MODE3), BT3.2, C1.2, J1.2, J1.3, P4.12 (P12), P5.4 (GND), P5.5 (shield), P6.4 (GND), P6.5 (shield), P9.1 (P1), P9.2 (P2), P9.3 (P3), P9.4 (P4), R1.2, U5.2 (VIN-), U5.4 (VOUT-)
- net at BT1.1, BT2.1: now also U3.21 (VBAT), BT3.1, SW3.2; no longer D2.1 (A)
- net at R2.1: now also U3.26 (PA1); no longer U3.33 (PB0)
- net at U2.4 (SDA), U3.36 (PB11): now also P2.2 (P2), U3.27 (PA2)
- net +5V: now reaches JP1.2, U3.18 (5V), U4.2 (5V), U4.4 (5V)
- net +5V: now also C1.1, P4.1 (VDD_5V), P5.1 (VCC), P6.1 (VCC), U5.3 (VOUT+)
- net at U3.7 (PA10): now also U1.7 (IO7/TXD), U4.10 (GPIO15/RXD)
- net at U1.6 (IO6/RXD), U4.8 (GPIO14/TXD): now also U3.6 (PA9); no longer U3.14 (PB6)
- net at U3.3 (PB14): now also R5.1
- net at U3.31 (PA6): now also P7.4 (P4)
- net at U3.32 (PA7): now also P7.3 (P3)
- net at U3.34 (PB1): now also P7.1 (P1)
- net at U3.4 (PB15): now also P3.1 (P1), R1.1
- net at U4.15 (GPIO22): now also R5.2
- new net: D2.1 (A), SW3.1
- new net: P7.2 (P2), U3.33 (PB0)
- new net: P4.2 (P2), P5.3 (D+)
- new net: P4.3 (P3), P5.2 (D-)
- new net: P4.4 (P4), P6.3 (D+)
- new net: P4.5 (P5), P6.2 (D-)
- new net +BATT: D2.2 (K), J1.1, JP1.1, P8.1 (P1), P8.2 (P2), P8.3 (P3), P8.4 (P4), R3.1, U1.23 (VCC), U3.20 (3.3V), U3.38 (3.3V), U5.1 (VIN+)
- now unconnected: U3.15 (PB7)
Other:
- moved on the sheet: BT1, BT2, SW2

Commit message: Change to Take 3
Parts:
- removed P3: EN, Pin_Headers:Pin_Header_Straight_1x01, symbol CONN_01X01
- added JP2, JP3: JUMPER3, Pin_Headers:Pin_Header_Straight_1x03, symbol JUMPER3
- added Q1: MOSFET_P, TO_SOT_Packages_SMD:SOT-23_Handsoldering, symbol MOSFET_P
- added U6: ES920LR_LPWA_EASEL, library:ES920_LPWA_EASEL, symbol ES920LR_LPWA_EASEL
- added W1, W2, W3: TEST_1P, Pin_Headers:Pin_Header_Straight_1x01, symbol TEST_1P
Connections:
- net +BATT: now also R1.2, Q1.D, U6.13 (VCC), U6.2 (VCCRF); no longer U5.1 (VIN+)
- net GND: now also U6.1 (GND), U6.26 (GND), U6.27 (GND); no longer R1.2
- net at U3.1 (PB12): now also U6.16 (PTC1/SW_INT)
- net at R1.1, U3.4 (PB15): now also Q1.G
- net at U1.6 (IO6/RXD), U3.6 (PA9): now also JP2.1, JP3.3, U6.9 (PTA1/UART0_RX); no longer U4.8 (GPIO14/TXD)
- net at U1.7 (IO7/TXD), U3.7 (PA10): now also JP2.3, JP3.1, U6.8 (PTA2/UART0_TX); no longer U4.10 (GPIO15/RXD)
- new net: JP3.2, U4.10 (GPIO15/RXD)
- new net: JP2.2, U4.8 (GPIO14/TXD)
- new net: Q1.S, U5.1 (VIN+)
- new net: U6.24 (RESETB), W3.1
- new net: U6.5 (PTA0/SWD_CLK), W1.1
- new net: U6.6 (PTA3/SWD_DIO), W2.1
- no-connect marks 63 -> 78
Other:
- moved on the sheet: J1, P4, P5, P6, R1, SP1
